File: hardware/fobos-mtc/fobos-mtc.kicad_pcb (KiCad board)
At the start: 2 copper layers, 76.2 x 40.6 mm, 52 parts, among them J1 Conn_01x10, J10 Conn_02x10_Odd_Even, J11 Conn_02x10_Odd_Even, J12 Conn_02x06_Top_Bottom, J13 Conn_02x06_Top_Bottom, J2 Conn_01x10, J3 Conn_01x10, J4 Conn_01x10, J5 Target, J6 Conn_01x02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

Commit message: restructuring TVGEN documentation, checking serial for MTC
Other:
- net class Default removed
