File: hardware/fobos-dut/dut-artix7-a12t-cpg238/User Button and IO.kicad_sch (KiCad schematic)
At the start: 26 parts, among them Q3 BSS138, Q4 BSS138, Q5 BSS138, Q6 BSS138

Commit message: cleaned up FBDA7 rev1 added BOM, fixed bugs in schematic
Parts:
- renumbered Q3 to Q4, Q4 to Q6, Q6 to Q7, R37 to R57, R40 to R58, R42 to R59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
