File: hardware/fobos-dut/dut-artix7-a12t-cpg238/fpga 1.kicad_sch (KiCad schematic)
At the start: 24 parts, among them U11 IS25LP256D-JMLE, U7 XC7A12T-CPG238

Commit message: cleaned up FBDA7 rev1 added BOM, fixed bugs in schematic
Parts:
- R77: renamed from R80; now not fitted
- renumbered C52 to C16, C40 to C25, C41 to C26, C42 to C27, C43 to C28, C44 to C29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
Other:
- note removed: "DNP"
