File: hardware/fobos-dut/dut-artix7-a12t-cpg238/fpgapower.kicad_sch (KiCad schematic)
At the start: 13 parts, among them U7 XC7A12T-CPG238

Commit message: cleaned up FBDA7 rev1 added BOM, fixed bugs in schematic
Parts:
- C38: renamed from C8; now not fitted
- C41: renamed from C12; now not fitted
- C42: renamed from C19; now not fitted
- C44: renamed from C16; now not fitted
- C46: renamed from C18; now not fitted
- C47: renamed from C14; now not fitted
- C55: renamed from C9; now not fitted
- C56: renamed from C13; now not fitted
- renumbered C10 to C39, C11 to C40, C15 to C43, C17 to C45, U7 to U1
