File: hardware/fobos-dut/dut-artix7-a12t-cpg238/fpgaprog.kicad_sch (KiCad schematic)
At the start: 13 parts, among them J7 0878321420, Q2 BSS138, SW1 SW_DIP_x03, U7 XC7A12T-CPG238

Commit message: cleaned up FBDA7 rev1 added BOM, fixed bugs in schematic
Parts:
- removed D8: LG_L29K-G2J1-24-Z, LED_SMD:LED_0603_1608Metric, symbol Device:LED
- removed Q2: BSS138, Package_TO_SOT_SMD:SOT-23, symbol Transistor_FET:BSS138
- removed R26: 470R, Resistor_SMD:R_0603_1608Metric, symbol Device:R
- added D6: LG_L29K-G2J1-24-Z, LED_SMD:LED_0603_1608Metric, symbol cerg:LG_L29K-G2J1-24-Z
- added R53, R72: 200R, Resistor_SMD:R_0603_1608Metric, symbol Device:R
- renumbered C7 to C37, R31 to R29, R27 to R31, R28 to R32, R29 to R33, R33 to R54, R34 to R55, U7 to U1
Connections:
- net +3V3: now also R53.2
- net GND: now also D6.2
- net SW_DONE: now also R53.1, R72.2
- new net: D6.1, R72.1
Other:
- note removed: "Configuration Mode SW1_0 SW1_1 SW1_2"
- note removed: "FLASH - Master SPI On On Off"
- note removed: "FOBOS - Slave Serial Off Off Off"
- note removed: "JTAG - JTAG Off On Off"
- note removed: "User LED_1"
